File: hardware/reloaded/MSX OPL4 Wozblaster.kicad_sch (KiCad schematic)
At the start: 48 parts

Commit message: conversion fixes
Parts:
- C1: value (none) -> 10pF; footprint (none) -> MSX OPL4 Wozblaster:C2.5-2
- C10, C9: value (none) -> 22uF; footprint (none) -> MSX OPL4 Wozblaster:E2,5-5
- C11, C4: value (none) -> 15nF; footprint (none) -> MSX OPL4 Wozblaster:C2.5-2
- C12, C2: value (none) -> 330nF; footprint (none) -> MSX OPL4 Wozblaster:C2.5-2
- C13, C16, C17, C18, C23: value (none) -> 100nF; footprint (none) -> MSX OPL4 Wozblaster:C2.5-2
- C14, C15: value (none) -> 12pF; footprint (none) -> MSX OPL4 Wozblaster:C2.5-2
- C19, C20: value (none) -> 100nf; footprint (none) -> MSX OPL4 Wozblaster:C2.5-2
- C21: value (none) -> 4.7uF; footprint (none) -> MSX OPL4 Wozblaster:E2,5-5
- C22: value (none) -> 470uF 16V; footprint (none) -> MSX OPL4 Wozblaster:D_7343-31R
- C3: value (none) -> 2200p; footprint (none) -> MSX OPL4 Wozblaster:C2.5-2
- C5, C6, C7: value (none) -> 2.2nF; footprint (none) -> MSX OPL4 Wozblaster:C2.5-2
- C8: value (none) -> 10uF; footprint (none) -> MSX OPL4 Wozblaster:E2,5-5
- IC1: value (none) -> OPL4_10X10; footprint (none) -> MSX OPL4 Wozblaster:OPL410X10
- IC2: value (none) -> YMF278B-F; footprint (none) -> MSX OPL4 Wozblaster:80-QFP
- IC3: value (none) -> YAC513-M; footprint (none) -> MSX OPL4 Wozblaster:16SOP
- IC4: value (none) -> DIL42; footprint (none) -> MSX OPL4 Wozblaster:DIL42
- IC5: value (none) -> ATF16V8BP3; footprint (none) -> MSX OPL4 Wozblaster:DIL20
- Q1: value (none) -> 33.8688; footprint (none) -> MSX OPL4 Wozblaster:HC49_S
- R1, R2: value (none) -> 360; footprint (none) -> MSX OPL4 Wozblaster:0204_7
- R10, R11, R12, R3, R4, R5, R8: value (none) -> 1k; footprint (none) -> MSX OPL4 Wozblaster:0204_7
- R13: value (none) -> 3.3k; footprint (none) -> MSX OPL4 Wozblaster:0204_7
- R6: value (none) -> 1K; footprint (none) -> MSX OPL4 Wozblaster:0204_7
- R7, R9: value (none) -> 100k; footprint (none) -> MSX OPL4 Wozblaster:0204_7
- U$1: value (none) -> 50PINCONN; footprint (none) -> MSX OPL4 Wozblaster:MSX50PINHEADER
- U$4, U$5: value (none) -> SRAM4MBIT; footprint (none) -> MSX OPL4 Wozblaster:SOP32L
- U$6: value (none) -> MSXJACK; footprint (none) -> MSX OPL4 Wozblaster:1501_06
- U2: renamed from U$2; value (none) -> LF347SO14; footprint (none) -> MSX OPL4 Wozblaster:SO14-2
- U3: renamed from U$3; value (none) -> LF347; footprint (none) -> MSX OPL4 Wozblaster:SO14-2
Connections:
- net A10: no longer U$5.23 (A10)
- no-connect marks 0 -> 6
Other:
- moved on the sheet: C10, C11, C12, C2, C20, C3, C4, C5, C9, R10, R11, R12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
