File: hardware/reloaded_v1.2/MSX OPL4 Wozblaster/MSX OPL4 Wozblaster.kicad_pcb (KiCad board)
At the start: 4 copper layers, 100 x 64.8 mm, 56 parts, among them IC1 LF347, IC2 GAL16V8D, IC3 KM684000ALG, IC4 LF347, IC5 KM684000ALG, IC6 YMF278B-F, IC7 YAC513-M, IC8 AM29F016B-120EC, J1 PJ-307, Q1 33.8688

Commit message: Uploading Gerbers vor v1.2
Parts:
- moved R11 1.27 mm to (215.1, 102.9)
- moved C17 0.84 mm to (214.6, 106.9)
Routing:
- net /A2: track 0.00 -> 111.5 mm, vias 0 -> 1
- net /~{ROM}: track 0.00 -> 110.1 mm, vias 0 -> 2
- net /A5: track 0.00 -> 98.3 mm, vias 0 -> 1
- net /A0: track 0.00 -> 94.1 mm, vias 0 -> 2
- net /MD5: track 0.00 -> 92.7 mm, vias 0 -> 2
- net /MD6: track 0.00 -> 91.5 mm, vias 0 -> 2
- net /A3: track 0.00 -> 89.3 mm, vias 0 -> 1
- net Net-(C13-+): track 0.00 -> 88.5 mm
- net /A1: track 0.00 -> 87.1 mm, vias 0 -> 3
- net Net-(IC1C-IN-): track 0.00 -> 85.5 mm
- net /A10: track 0.00 -> 85.4 mm, vias 0 -> 4
- net /A4: track 0.00 -> 85.2 mm, vias 0 -> 3
- net /MD4: track 0.00 -> 80.8 mm, vias 0 -> 2
- net GND: track 0.00 -> 80.1 mm, vias 0 -> 34
- net /A9: track 0.00 -> 72.3 mm, vias 0 -> 3
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