File: hardware/reloaded_v2.1/MSX OPL4 Wozblaster/MSX OPL4 Wozblaster.kicad_pcb (KiCad board)
At the start: 4 copper layers, 100 x 64.8 mm, 64 parts, among them IC1 GAL16V8D, IC2 KM684000ALG, IC3 KM684000ALG, IC4 YMF278B-F, IC5 AM29F016B-120EC, J1 PJ-307, Q1 33.8688, T1 2SA733, T2 2SC945, T3 2SC945, T4 2SC945, U1 NJM4558, U2 NJM4558, U3 uPD6376

Commit message: v3 and multiple adjusts
Parts:
- U1, U2: footprint Package_SO:MSOP-8_3x3mm_P0.65mm -> Package_SO:SO-8_5.3x6.2mm_P1.27mm
- moved C16 3.61 mm to (153.9, 112.0)
- moved C15 2.21 mm to (143.2, 115.7), turned to 0 degrees
Routing:
- net GND: track 52.3 -> 72.9 mm
- net +5V: track 45.4 -> 54.8 mm
- net Net-(U1A-+): track 72.4 -> 76.4 mm
- net Net-(C4-+): track 34.1 -> 37.6 mm
- net Net-(C20--): track 14.8 -> 17.1 mm
- net /MD6: track 49.6 -> 50.7 mm
- net Net-(C24-+): track 18.7 -> 19.5 mm
- net Net-(C25-+): track 19.2 -> 18.5 mm
- net Net-(U1A--): track 7.68 -> 7.04 mm
- net Net-(C21--): track 15.2 -> 15.7 mm
Other:
- board text added: "v2.1"
- board text removed: "v2.0"
